File: RC-PT1/RC-PT1.kicad_pcb (KiCad board)
At the start: 2 copper layers, 100 x 100 mm, 13 parts

Commit message: remove DT1
Parts:
- removed the G*** at (115.0, 111.0)
Other:
- outline, holes or cut-outs redrawn
- board text added: "Pasivni RC krug"
- board text removed: "Pasivni RC krug - PT1 član"
- board text removed: "U₁"
- board text removed: "U₂"
