File: RC-PT1/RC-PT1.kicad_pcb (KiCad board)
At the start: 2 copper layers, 100 x 100 mm, 16 parts

Commit message: Fix libraries
Parts:
- removed TP5, TP6, TP7, TP8: TestPoint_Alt, Library:KEYS4952
Routing:
- net Net-(C1-Pad2): track 133.9 -> 121.9 mm
- net Net-(R1-Pad1): track 49.4 -> 43.4 mm
- net Net-(C1-Pad1): track 86.9 -> 80.9 mm

Commit message: Logos
Parts:
- removed the G*** at (146.0, 64.0)
- added G***: LOGO, Library:tvz, F.Cu at (175.5, 150.0)
- moved TP1 2.00 mm to (107.5, 73.5)
- moved TP2 2.00 mm to (107.5, 138.0)
- moved TP3 2.00 mm to (184.5, 74.0)
- moved TP4 2.00 mm to (184.5, 138.0)
Connections:
- net Net-(C1-Pad2) renamed GND
Routing:
- net Net-(R1-Pad1): track 43.4 -> 36.3 mm
- net Net-(C1-Pad1): track 80.9 -> 74.7 mm
- net GND: track 121.9 -> 120.4 mm
- added copper zone on F.Cu, net GND

Commit message: PI
Changed lines of the file:
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@@
 	(gr_circle
 		(center 100 60)
-		(end 103 60)
+		(end 103.1 60)
 		(stroke
 			(width 0.2)
@@
 	(gr_circle
 		(center 100 152)
-		(end 103 152)
+		(end 103.1 152)
 		(stroke
 			(width 0.2)
@@
 	(gr_circle
 		(center 192 60)
-		(end 195 60)
+		(end 195.1 60)
 		(stroke
 			(width 0.2)
@@
 	(gr_circle
 		(center 192 152)
-		(end 195 152)
+		(end 195.1 152)
 		(stroke
 			(width 0.2)
@@
 	)
 	(segment
+		(start 167.85 129)
+		(end 176.85 138)
+		(width 1)
+		(layer "B.Cu")
+		(net "GND")
+	)
+	(segment
+		(start 154.5 129)
+		(end 124.15 129)
+		(width 1)
+		(layer "B.Cu")
+		(net "GND")
+	)
+	(segment
+		(start 115.15 138)
+		(end 99.85 138)
+		(width 3)
+		(layer "B.Cu")
+		(net "GND")
+	)
+	(segment
+		(start 192.15 138)
+		(end 176.85 138)
+		(width 3)
+		(layer "B.Cu")
+		(net "GND")
+	)
+	(segment
+		(start 124.15 129)
+		(end 115.15 138)
+		(width 1)
+		(layer "B.Cu")
+		(net "GND")
+	)
+	(segment
+		(start 154.5 129)
+		(end 167.85 129)
+		(width 1)
+		(layer "B.Cu")
+		(net "GND")
+	)
+	(segment
+		(start 115.25 140)
+		(end 115.15 140)
+		(width 1)
+		(layer "B.Cu")
+		(net "GND")
+	)
+	(segment
+		(start 154.5 129)
+		(end 154.5 108.5)
+		(width 1)
+		(layer "B.Cu")
+		(net "GND")
+	)
+	(segment
 		(start 99.85 73.5)
 		(end 115.15 73.5)
@@
 		(layer "B.Cu")
 		(net "Net-(R1-Pad1)")
-	)
-	(segment
-		(start 167.85 129)
-		(end 176.85 138)
-		(width 1)
-		(layer "B.Cu")
-		(net "GND")
-	)
-	(segment
-		(start 154.5 129)
-		(end 124.15 129)
-		(width 1)
-		(layer "B.Cu")
-		(net "GND")
-	)
-	(segment
-		(start 115.15 138)
-		(end 99.85 138)
-		(width 3)
-		(layer "B.Cu")
-		(net "GND")
-	)
-	(segment
-		(start 192.15 138)
-		(end 176.85 138)
-		(width 3)
-		(layer "B.Cu")
-		(net "GND")
-	)
-	(segment
-		(start 124.15 129)
-		(end 115.15 138)
-		(width 1)
-		(layer "B.Cu")
-		(net "GND")
-	)
-	(segment
-		(start 154.5 129)
-		(end 167.85 129)
-		(width 1)
-		(layer "B.Cu")
-		(net "GND")
-	)
-	(segment
-		(start 115.25 140)
-		(end 115.15 140)
-		(width 1)
-		(layer "B.Cu")
-		(net "GND")
-	)
-	(segment
-		(start 154.5 129)
-		(end 154.5 108.5)
-		(width 1)
-		(layer "B.Cu")
-		(net "GND")
 	)
 	(zone
@@
 			)
 		)
+	)
+	(zone
+		(layers "F.Cu" "B.Cu")
+		(hatch edge 0.5)
+		(connect_pads
+			(clearance 0)
+		)
+		(min_thickness 0.25)
+		(keepout
+			(tracks allowed)
+			(vias allowed)
+			(pads allowed)
+			(copperpour not_allowed)
+			(footprints allowed)
+		)
+		(placement
+			(enabled no)
+			(sheetname "")
+		)
+		(fill
+			(thermal_gap 0.5)
+			(thermal_bridge_width 0.5)
+			(island_removal_mode 0)
+		)
+		(polygon
+			(pts
+				(arc
+					(start 97 60)
+					(mid 103 60)
+					(end 97 60)
+				)
+			)
+		)
+	)
+	(zone
+		(layers "F.Cu" "B.Cu")
+		(hatch edge 0.5)
+		(connect_pads
+			(clearance 0)
+		)
+		(min_thickness 0.25)
+		(keepout
+			(tracks allowed)
+			(vias allowed)
+			(pads allowed)
+			(copperpour not_allowed)
+			(footprints allowed)
+		)
+		(placement
+			(enabled no)
+			(sheetname "")
+		)
+		(fill
+			(thermal_gap 0.5)
+			(thermal_bridge_width 0.5)
+			(island_removal_mode 0)
+		)
+		(polygon
+			(pts
+				(arc
+					(start 97 152)
+					(mid 103 152)
+					(end 97 152)
+				)
+			)
+		)
+	)
+	(zone
+		(layers "F.Cu" "B.Cu")
+		(hatch edge 0.5)
+		(connect_pads
+			(clearance 0)
+		)
+		(min_thickness 0.25)
+		(keepout
+			(tracks allowed)
+			(vias allowed)
+			(pads allowed)
+			(copperpour not_allowed)
+			(footprints allowed)
+		)
+		(placement
+			(enabled no)
+			(sheetname "")
+		)
+		(fill
+			(thermal_gap 0.5)
+			(thermal_bridge_width 0.5)
+			(island_removal_mode 0)
+		)
+		(polygon
+			(pts
+				(arc
+					(start 189 152)
+					(mid 195 152)
+					(end 189 152)
+				)
+			)
+		)
+	)
+	(zone
+		(layers "F.Cu" "B.Cu")
+		(hatch edge 0.5)
+		(connect_pads
+			(clearance 0)
+		)
+		(min_thickness 0.25)
+		(keepout
+			(tracks allowed)
+			(vias allowed)
+			(pads allowed)
+			(copperpour not_allowed)
+			(footprints allowed)
+		)
+		(placement
+			(enabled no)
+			(sheetname "")
+		)
+		(fill
+			(thermal_gap 0.5)
+			(thermal_bridge_width 0.5)
+			(island_removal_mode 0)
+		)
+		(polygon
+			(pts
+				(arc
+					(start 189 60)
+					(mid 195 60)
+					(end 189 60)
+				)
+			)
+		)
