File: RC-PT1/RC-PT1.kicad_sch (KiCad schematic)
At the start: 10 parts

Commit message: Dodan aktivni član PT1/DT1
Parts:
- added TP5, TP6, TP7, TP8: TestPoint_Alt, Library:KEYS4952, symbol Connector:TestPoint_Alt
Connections:
- net at R1.1, TP1.1: now also TP5.1
- net at C1.1, R1.2, TP3.1: now also TP6.1
- net at C1.2, TP2.1, TP4.1: now also TP7.1, TP8.1

Commit message: Fix libraries
Parts:
- removed TP5, TP6, TP7, TP8: TestPoint_Alt, Library:KEYS4952, symbol Connector:TestPoint_Alt

Commit message: Logos
Parts:
- C1: TME (none) -> R82DC4100DQ60J
Connections:
- net GND: now reaches C1.2, TP2.1, TP4.1
Other:
- note added: "RC krug"
- note removed: "PT1"
Changed lines of the file:
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@@
 	(generator_version "10.0")
 	(paper "A4")
-	(text "PT1"
+	(text "RC krug"
 		(exclude_from_sim no)
 		(at 137.16 67.31 0)
@@
 	)
 	(junction
+		(at 116.84 96.52)
+		(diameter 0)
+		(color 0 0 0 0)
+	)
+	(junction
 		(at 137.16 77.47)
 		(diameter 0)
@@
 	(wire
 		(pts
-			(xy 113.03 96.52) (xy 137.16 96.52)
+			(xy 113.03 96.52) (xy 116.84 96.52)
 		)
 		(stroke
@@
 	(wire
 		(pts
-			(xy 127 77.47) (xy 137.16 77.47)
+			(xy 116.84 96.52) (xy 116.84 100.33)
 		)
 		(stroke
@@
 	(wire
 		(pts
-			(xy 137.16 77.47) (xy 137.16 82.55)
+			(xy 127 77.47) (xy 137.16 77.47)
 		)
 		(stroke
@@
 	(wire
 		(pts
-			(xy 113.03 77.47) (xy 119.38 77.47)
+			(xy 137.16 77.47) (xy 137.16 82.55)
 		)
 		(stroke
@@
 	(wire
 		(pts
+			(xy 113.03 77.47) (xy 119.38 77.47)
+		)
+		(stroke
+			(width 0)
+			(type default)
+		)
+	)
+	(wire
+		(pts
 			(xy 137.16 96.52) (xy 152.4 96.52)
+		)
+		(stroke
+			(width 0)
+			(type default)
+		)
+	)
+	(wire
+		(pts
+			(xy 116.84 96.52) (xy 137.16 96.52)
 		)
 		(stroke
@@
 			)
 		)
+		(property "TME" ""
+			(at 148.59 181.61 0)
+			(hide yes)
+			(show_name no)
+			(do_not_autoplace no)
+			(effects
+				(font
+					(size 1.27 1.27)
+				)
+			)
+		)
 		(instances
 			(project "RC-PT1"
@@
 			)
 		)
+		(property "TME" ""
+			(at 123.19 77.47 90)
+			(hide yes)
+			(show_name no)
+			(do_not_autoplace no)
+			(effects
+				(font
+					(size 1.27 1.27)
+				)
+			)
+		)
 		(pin "1"
 		)
@@
 			)
 		)
+		(property "TME" ""
+			(at 148.59 186.69 0)
+			(hide yes)
+			(show_name no)
+			(do_not_autoplace no)
+			(effects
+				(font
+					(size 1.27 1.27)
+				)
+			)
+		)
 		(instances
 			(project "RC-PT1"
@@
 			)
 		)
+		(property "TME" ""
+			(at 113.03 96.52 90)
+			(hide yes)
+			(show_name no)
+			(do_not_autoplace no)
+			(effects
+				(font
+					(size 1.27 1.27)
+				)
+			)
+		)
 		(pin "1"
 		)
@@
 			)
 		)
+		(property "TME" ""
+			(at 152.4 96.52 90)
+			(hide yes)
+			(show_name no)
+			(do_not_autoplace no)
+			(effects
+				(font
+					(size 1.27 1.27)
+				)
+			)
+		)
 		(pin "1"
 		)
@@
 			)
 		)
+		(property "TME" ""
+			(at 152.4 77.47 90)
+			(hide yes)
+			(show_name no)
+			(do_not_autoplace no)
+			(effects
+				(font
+					(size 1.27 1.27)
+				)
+			)
+		)
 		(pin "1"
 		)
@@
 			)
 		)
+		(property "TME" ""
+			(at 148.59 171.45 0)
+			(hide yes)
+			(show_name no)
+			(do_not_autoplace no)
+			(effects
+				(font
+					(size 1.27 1.27)
+				)
+			)
+		)
 		(instances
 			(project "RC-PT1"
@@
 			)
 		)
+		(property "TME" ""
+			(at 113.03 77.47 90)
+			(hide yes)
+			(show_name no)
+			(do_not_autoplace no)
+			(effects
+				(font
+					(size 1.27 1.27)
+				)
+			)
+		)
 		(pin "1"
 		)
@@
 				(path "/516af16e-4df2-44b9-98db-abada191c38c"
 					(reference "TP1")
+					(unit 1)
+				)
+			)
+		)
+	)
+	(symbol
+		(lib_id "power:GND")
+		(at 116.84 100.33 0)
+		(unit 1)
+		(body_style 1)
+		(exclude_from_sim no)
+		(in_bom yes)
+		(on_board yes)
+		(in_pos_files yes)
+		(dnp no)
+		(fields_autoplaced yes)
+		(property "Reference" "#PWR01"
+			(at 116.84 106.68 0)
+			(hide yes)
+			(show_name no)
+			(do_not_autoplace no)
+			(effects
+				(font
+					(size 1.27 1.27)
+				)
+			)
+		)
+		(property "Value" "GND"
+			(at 116.84 105.41 0)
+			(show_name no)
+			(do_not_autoplace no)
+			(effects
+				(font
+					(size 1.27 1.27)
+				)
+			)
+		)
+		(property "Footprint" ""
+			(at 116.84 100.33 0)
+			(hide yes)
+			(show_name no)
+			(do_not_autoplace no)
+			(effects
+				(font
+					(size 1.27 1.27)
+				)
+			)
+		)
+		(property "Datasheet" ""
+			(at 116.84 100.33 0)
+			(hide yes)
+			(show_name no)
+			(do_not_autoplace no)
+			(effects
+				(font
+					(size 1.27 1.27)
+				)
+			)
+		)
+		(property "Description" "Power symbol creates a global label with name \"GND\" , ground"
+			(at 116.84 100.33 0)
+			(hide yes)
+			(show_name no)
+			(do_not_autoplace no)
+			(effects
+				(font
+					(size 1.27 1.27)
+				)
+			)
+		)
+		(pin "1"
+		)
+		(instances
+			(project "RC-PT1"
+				(path "/516af16e-4df2-44b9-98db-abada191c38c"
+					(reference "#PWR01")
 					(unit 1)
 				)
@@
 			)
 		)
+		(property "TME" ""
+			(at 148.59 176.53 0)
+			(hide yes)
+			(show_name no)
+			(do_not_autoplace no)
+			(effects
+				(font
+					(size 1.27 1.27)
+				)
+			)
+		)
 		(instances
 			(project "RC-PT1"
@@
 			(at 137.16 86.36 0)
 			(hide yes)
+			(show_name no)
+			(do_not_autoplace no)
+			(effects
+				(font
+					(size 1.27 1.27)
+				)
+			)
+		)
+		(property "TME" "R82DC4100DQ60J"
+			(at 137.16 86.36 0)
+			(hide yes)
