File: Active-PT1-DT1/Active-PT1-DT1.kicad_sch (KiCad schematic)
At the start: 27 parts, among them U1 Opamp_Dual

Commit message: PT1/DT1/P
Parts:
- removed TP5, TP6, TP7, TP8: TestPoint_Alt, Library:KEYS4952, symbol Connector:TestPoint_Alt
- removed U1: Opamp_Dual, Package_DIP:DIP-8_W7.62mm_Socket_LongPads, symbol Device:Opamp_Dual
- added U1: TL072, Package_DIP:DIP-8_W7.62mm_LongPads, symbol Amplifier_Operational:TL072
- C1, C2: footprint Capacitor_THT:C_Rect_L7.2mm_W5.0mm_P5.00mm -> (none)
- R6: value 50k -> 47k; now not fitted
Connections:
- net at C1.2, JP1.3 (B), JP2.1 (A)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: now also U1.2 (-)
- net at C2.2, R2.2, R4.1: now also U1.1
- net at TP9.1: now also U1.8 (V+)
- net at R6.2: now also U1.5 (+)
- net at R5.2, TP3.1: now also U1.7
- net at R4.2, R5.1: now also U1.6 (-)
- net at R3.2: now also U1.3 (+)
- net at D1.2 (A): now also U1.4 (V-)
Other:
- moved on the sheet: C1, C2, D1, JP1, JP2, R1, TP1, TP10, TP11, TP2, TP9

Commit message: Fix libraries
Parts:
- JP1, JP2: footprint Connector_PinHeader_2.54mm:PinHeader_1x03_P2.54mm_Vertical -> Library:Jumper_1x03
- R6: now fitted
- TP11: footprint Library:DELTRON 4mm banana socket - black -> Library:DELTRON 4mm banana socket - blue
- TP9: footprint Library:DELTRON 4mm banana socket - black -> Library:DELTRON 4mm banana socket - yellow
Changed lines of the file:
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@@
 			)
 		)
-		(property "Footprint" "Library:DELTRON 4mm banana socket - black"
+		(property "Footprint" "Library:DELTRON 4mm banana socket - yellow"
 			(at 107.95 123.19 0)
 			(hide yes)
@@
 		(on_board yes)
 		(in_pos_files yes)
-		(dnp yes)
+		(dnp no)
 		(property "Reference" "R6"
 			(at 167.64 88.9 90)
@@
 		(fields_autoplaced yes)
 		(property "Reference" "JP1"
-			(at 106.68 57.15 0)
+			(at 106.68 59.69 0)
 			(show_name no)
 			(do_not_autoplace no)
@@
 		(property "Value" "Jumper_3_Open"
 			(at 106.68 59.69 0)
-			(show_name no)
-			(do_not_autoplace no)
-			(effects
-				(font
-					(size 1.27 1.27)
-				)
-			)
-		)
-		(property "Footprint" "Connector_PinHeader_2.54mm:PinHeader_1x03_P2.54mm_Vertical"
+			(hide yes)
+			(show_name no)
+			(do_not_autoplace no)
+			(effects
+				(font
+					(size 1.27 1.27)
+				)
+			)
+		)
+		(property "Footprint" "Library:Jumper_1x03"
 			(at 106.68 63.5 0)
 			(hide yes)
@@
 			)
 		)
-		(property "Footprint" "Library:DELTRON 4mm banana socket - black"
+		(property "Footprint" "Library:DELTRON 4mm banana socket - blue"
 			(at 97.79 146.05 0)
 			(hide yes)
@@
 		(fields_autoplaced yes)
 		(property "Reference" "JP2"
-			(at 130.81 50.8 0)
+			(at 130.81 53.34 0)
 			(show_name no)
 			(do_not_autoplace no)
@@
 		(property "Value" "Jumper_3_Open"
 			(at 130.81 53.34 0)
-			(show_name no)
-			(do_not_autoplace no)
-			(effects
-				(font
-					(size 1.27 1.27)
-				)
-			)
-		)
-		(property "Footprint" "Connector_PinHeader_2.54mm:PinHeader_1x03_P2.54mm_Vertical"
+			(hide yes)
+			(show_name no)
+			(do_not_autoplace no)
+			(effects
+				(font
+					(size 1.27 1.27)
+				)
+			)
+		)
+		(property "Footprint" "Library:Jumper_1x03"
 			(at 130.81 57.15 0)
 			(hide yes)

Commit message: PT1/DT1/P complete
Parts:
- removed D1: D_Schottky, symbol Device:D_Schottky
- added C3, C4: 0.1uF, Capacitor_THT:C_Rect_L7.2mm_W2.5mm_P5.00mm, symbol Device:C
- added D1, D2: 1N4007, Diode_THT:D_DO-41_SOD81_P10.16mm_Horizontal, symbol Diode:1N4007
- added F1, F2: 100mA, Capacitor_THT:C_Disc_D7.5mm_W4.4mm_P5.00mm, symbol Device:Polyfuse
- added TP5: TestPoint, Library:DELTRON 4mm banana socket - red, symbol Connector:TestPoint
- C1: footprint (none) -> Capacitor_THT:C_Rect_L7.2mm_W2.5mm_P5.00mm; TME (none) -> R82DC3100DQ50J
- C2: footprint (none) -> Capacitor_THT:C_Rect_L7.2mm_W2.5mm_P5.00mm; TME (none) -> R82EC2100AA50J
- TP1, TP3: TME (none) -> 571-0500
- TP10, TP2, TP4: TME (none) -> 571-0100
- TP11: TME (none) -> 571-0200
- TP9: TME (none) -> 571-0700
- U1: TME (none) -> TL072CP
Connections:
- net at C2.2, R2.2, R4.1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: now also TP5.1
- net at U1.4 (V-): now also C4.2, D2.2 (A), F2.2
- net at U1.8 (V+): now also C3.1, D1.1 (K), F1.2; no longer TP9.1
- net GND: now reaches R3.1, R6.1, TP10.1, TP2.1, TP4.1
- net GND: now also C3.2, C4.1, D1.2 (A), D2.1 (K)
- net at TP11.1: now also F2.1
- new net: F1.1, TP9.1
Other:
- moved on the sheet: TP11, TP9, U1C
