File: Active-PT1-DT1/Active-PT1-DT1.kicad_pcb (KiCad board)
At the start: 2 copper layers, 100 x 100 mm, 16 parts

Commit message: Dodan aktivni član PT1/DT1
Parts:
- added C2: 10nF, Capacitor_THT:C_Rect_L7.2mm_W5.0mm_P5.00mm, F.Cu at (137.7, 125.0)
- added JP1: Jumper_3_Open, Connector_PinHeader_2.54mm:PinHeader_1x03_P2.54mm_Vertical, F.Cu at (138.1, 114.4)
- added JP2: Jumper_3_Open, Connector_PinHeader_2.54mm:PinHeader_1x03_P2.54mm_Vertical, F.Cu at (142.7, 114.4)
- added R2: 100k, Resistor_THT:R_Axial_DIN0207_L6.3mm_D2.5mm_P10.16mm_Horizontal, F.Cu at (137.4, 94.2)
- added R3: 100k, Resistor_THT:R_Axial_DIN0207_L6.3mm_D2.5mm_P10.16mm_Horizontal, F.Cu at (137.4, 98.2)
- added TP10: TestPoint, Library:DELTRON 4mm banana socket - black, F.Cu at (146.0, 67.8)
- added TP11: TestPoint, Library:DELTRON 4mm banana socket - black, F.Cu at (158.0, 68.0)
- added TP9: TestPoint, Library:DELTRON 4mm banana socket - black, F.Cu at (134.0, 67.8)
- added U1: Opamp_Dual, Package_DIP:DIP-8_W7.62mm_Socket_LongPads, F.Cu at (137.9, 102.4)
- C1: value C -> 0.1uF
- R1: value R -> 10k
- moved G*** 91.3 mm to (120.0, 151.5)
Connections:
- C1 pad 1: Net-(C1-Pad1) -> Net-(JP1-A)
- C1 pad 2: Net-(C1-Pad2) -> Net-(JP1-C)
- R1 pad 2: Net-(C1-Pad1) -> Net-(JP1-A)
- TP2 pad 1: Net-(C1-Pad2) -> Net-(R3-Pad1)
- TP3 pad 1: Net-(C1-Pad1) -> Net-(C2-Pad2)
- TP4 pad 1: Net-(C1-Pad2) -> Net-(R3-Pad1)
- TP6 pad 1: Net-(C1-Pad1) -> Net-(C2-Pad2)
- TP7 pad 1: Net-(C1-Pad2) -> Net-(R3-Pad1)
- TP8 pad 1: Net-(C1-Pad2) -> Net-(R3-Pad1)
Routing:
- net Net-(C1-Pad2): track 133.9 -> 0.00 mm
- net Net-(C1-Pad1): track 86.9 -> 0.00 mm
- net Net-(R1-Pad1): track 49.4 -> 0.00 mm
Other:
- board text added: "PT1/DT1"
- board text removed: "C=1µF"
- board text removed: "R=1kΩ"
- board text removed: "RC krug"

Commit message: PT1/DT1/P
Parts:
- removed TP5, TP6, TP7, TP8: TestPoint_Alt, Library:KEYS4952
- added R4: 100k, Resistor_THT:R_Axial_DIN0207_L6.3mm_D2.5mm_P10.16mm_Horizontal, F.Cu at (113.6, 98.5)
- added R5: 100k, Resistor_THT:R_Axial_DIN0207_L6.3mm_D2.5mm_P10.16mm_Horizontal, F.Cu at (113.6, 102.6)
- added R6: 47k, Resistor_THT:R_Axial_DIN0207_L6.3mm_D2.5mm_P10.16mm_Horizontal, F.Cu at (113.6, 106.6)
- U1: value Opamp_Dual -> TL072; footprint Package_DIP:DIP-8_W7.62mm_Socket_LongPads -> Package_DIP:DIP-8_W7.62mm_LongPads
- moved U1 25.3 mm to (114.0, 110.7)
Connections:
- C1 pad 2: Net-(JP1-C) -> Net-(JP1-B)
- C2 pad 1: Net-(JP2-C) -> Net-(JP2-B)
- JP1 pad 2: Net-(JP1-C) -> Net-(JP1-A)
- JP1 pad 3: unconnected-(JP1-B-Pad3) -> Net-(JP1-B)
- JP2 pad 1: Net-(JP1-C) -> Net-(JP1-B)
- JP2 pad 2: Net-(JP2-C) -> Net-(JP1-B)
- JP2 pad 3: unconnected-(JP2-B-Pad3) -> Net-(JP2-B)
- R2 pad 1: Net-(JP1-C) -> Net-(JP1-B)
- TP3 pad 1: Net-(C2-Pad2) -> Net-(R5-Pad2)
- U1 pad 2: Net-(JP1-C) -> Net-(JP1-B)
- U1 pad 5: unconnected-(U1B-+-Pad5) -> Net-(U1B-+)
- U1 pad 6: unconnected-(U1B---Pad6) -> Net-(U1B--)
- U1 pad 7: unconnected-(U1-Pad7) -> Net-(R5-Pad2)
Other:
- board text added: "PT1/DT1/P"
- board text removed: "PT1/DT1"

Commit message: Fix libraries
Parts:
- JP1, JP2: footprint Connector_PinHeader_2.54mm:PinHeader_1x03_P2.54mm_Vertical -> Library:Jumper_1x03
- TP11: footprint Library:DELTRON 4mm banana socket - black -> Library:DELTRON 4mm banana socket - blue
- TP9: footprint Library:DELTRON 4mm banana socket - black -> Library:DELTRON 4mm banana socket - yellow
- moved R1 33.8 mm to (163.4, 96.0)
- moved TP9 31.5 mm to (165.5, 67.3)
- moved TP11 31.0 mm to (127.0, 67.3)
- moved TP1 2.00 mm to (107.5, 73.5)
- moved TP2 2.00 mm to (107.5, 138.0)
- moved TP3 2.00 mm to (184.5, 74.0)
- moved TP4 2.00 mm to (184.5, 138.0)
- moved TP10 0.56 mm to (146.2, 67.3)
Other:
- board text added: "+15V"
- board text added: "-15V"
- board text added: "GND"
- board text removed: "PT1/DT1/P"

Commit message: PT1/DT1/P complete
Parts:
- removed the G*** at (120.0, 151.5)
- added C3: 0.1uF, Capacitor_THT:C_Rect_L7.2mm_W2.5mm_P5.00mm, F.Cu at (155.7, 91.0)
- added C4: 0.1uF, Capacitor_THT:C_Rect_L7.2mm_W2.5mm_P5.00mm, F.Cu at (141.3, 91.0)
- added D1: 1N4007, Diode_THT:D_DO-41_SOD81_P10.16mm_Horizontal, F.Cu at (158.3, 97.0)
- added D2: 1N4007, Diode_THT:D_DO-41_SOD81_P10.16mm_Horizontal, F.Cu at (143.9, 97.0)
- added F1: 100mA, Capacitor_THT:C_Disc_D7.5mm_W4.4mm_P5.00mm, F.Cu at (167.8, 97.0)
- added F2: 100mA, Capacitor_THT:C_Disc_D7.5mm_W4.4mm_P5.00mm, F.Cu at (124.2, 97.0)
- added TP5: TestPoint, Library:DELTRON 4mm banana socket - red, F.Cu at (184.3, 74.0)
- C1, C2: footprint Capacitor_THT:C_Rect_L7.2mm_W5.0mm_P5.00mm -> Capacitor_THT:C_Rect_L7.2mm_W2.5mm_P5.00mm
- moved R6 64.6 mm to (177.5, 116.0), turned to -90 degrees
- moved R5 60.9 mm to (169.7, 126.2), turned to 90 degrees
- moved R1 60.3 mm to (107.0, 117.3)
- moved R4 47.5 mm to (160.2, 107.6)
- moved U1 40.9 mm to (154.4, 117.3)
- moved C1 33.2 mm to (124.2, 117.3), turned to 0 degrees
- moved R3 26.7 mm to (136.1, 124.9)
- moved R2 23.1 mm to (136.1, 117.3)
- moved C2 20.7 mm to (148.9, 107.6)
- moved TP3 19.0 mm to (184.3, 93.0)
- moved JP1 15.5 mm to (124.2, 107.6), turned to 90 degrees
- moved JP2 9.05 mm to (136.7, 107.6), turned to 90 degrees
- moved TP4 0.52 mm to (184.3, 138.5)
Connections:
- net Net-(R3-Pad1) renamed GND
- TP9 pad 1: Net-(U1C-V+) -> Net-(F1-Pad1)
- U1 pad 8: Net-(U1C-V+) -> Net-(D1-K)
Routing:
- net Net-(C2-Pad2): track 0.00 -> 102.6 mm
- net Net-(D2-A): track 0.00 -> 90.6 mm
- net Net-(R1-Pad1): track 0.00 -> 62.4 mm
- net Net-(R5-Pad2): track 0.00 -> 52.3 mm
- net Net-(JP1-B): track 0.00 -> 49.4 mm
- net Net-(F2-Pad1): track 0.00 -> 38.4 mm
- net Net-(D1-K): track 0.00 -> 33.1 mm
- net Net-(U1B--): track 0.00 -> 32.0 mm
- net Net-(F1-Pad1): track 0.00 -> 22.9 mm
- net Net-(JP1-A): track 0.00 -> 20.4 mm
- net Net-(U1B-+): track 0.00 -> 18.4 mm
- net Net-(U1A-+): track 0.00 -> 9.16 mm
- net Net-(JP2-B): track 0.00 -> 7.03 mm
- added copper zone on B.Cu, net GND
- added copper zone on F.Cu, net GND
Other:
- board text added: "COM"
- board text added: "INV. IZLAZ"
- board text added: "NEINV.IZLAZ"
- board text added: "ULAZ"

Commit message: Update Active-PT1-DT1.kicad_pcb
Other:
- board text added: "0.1µF"
- board text added: "100k"
- board text added: "10k"
- board text added: "10nF"
- board text added: "47k"
- board text added: "TL072"
- board text removed: "COM"
