File: Active-PT1-DT1/Active-PT1-DT1.kicad_pcb (KiCad board)
At the start: 2 copper layers, 100 x 100 mm, 31 parts, among them U1 TL072

Commit message: PI
Changed lines of the file:
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@@
 	(gr_circle
 		(center 100 60)
-		(end 103 60)
+		(end 103.1 60)
 		(stroke
 			(width 0.2)
@@
 	(gr_circle
 		(center 100 152)
-		(end 103 152)
+		(end 103.1 152)
 		(stroke
 			(width 0.2)
@@
 	(gr_circle
 		(center 192 60)
-		(end 195 60)
+		(end 195.1 60)
 		(stroke
 			(width 0.2)
@@
 	(gr_circle
 		(center 192 152)
-		(end 195 152)
+		(end 195.1 152)
 		(stroke
 			(width 0.2)
@@
 			(header yes)
 			(stroke
-				(width 0.1)
+				(width 0.2)
 				(type solid)
 			)
@@
 			(cols yes)
 			(stroke
-				(width 0.1)
+				(width 0.2)
 				(type solid)
 			)
@@
 	)
 	(zone
+		(layers "F.Cu" "B.Cu")
+		(hatch edge 0.5)
+		(connect_pads
+			(clearance 0)
+		)
+		(min_thickness 0.25)
+		(keepout
+			(tracks allowed)
+			(vias allowed)
+			(pads allowed)
+			(copperpour not_allowed)
+			(footprints allowed)
+		)
+		(placement
+			(enabled no)
+			(sheetname "")
+		)
+		(fill
+			(thermal_gap 0.5)
+			(thermal_bridge_width 0.75)
+			(island_removal_mode 0)
+		)
+		(polygon
+			(pts
+				(arc
+					(start 97 152)
+					(mid 103 152)
+					(end 97 152)
+				)
+			)
+		)
+	)
+	(zone
+		(layers "F.Cu" "B.Cu")
+		(hatch edge 0.5)
+		(connect_pads
+			(clearance 0)
+		)
+		(min_thickness 0.25)
+		(keepout
+			(tracks allowed)
+			(vias allowed)
+			(pads allowed)
+			(copperpour not_allowed)
+			(footprints allowed)
+		)
+		(placement
+			(enabled no)
+			(sheetname "")
+		)
+		(fill
+			(thermal_gap 0.5)
+			(thermal_bridge_width 0.75)
+			(island_removal_mode 0)
+		)
+		(polygon
+			(pts
+				(arc
+					(start 97 60)
+					(mid 103 60)
+					(end 97 60)
+				)
+			)
+		)
+	)
+	(zone
 		(net "GND")
 		(layers "F.Cu" "B.Cu")
@@
 			)
 		)
+	)
+	(zone
+		(layers "F.Cu" "B.Cu")
+		(hatch edge 0.5)
+		(connect_pads
+			(clearance 0)
+		)
+		(min_thickness 0.25)
+		(keepout
+			(tracks allowed)
+			(vias allowed)
+			(pads allowed)
+			(copperpour not_allowed)
+			(footprints allowed)
+		)
+		(placement
+			(enabled no)
+			(sheetname "")
+		)
+		(fill
+			(thermal_gap 0.5)
+			(thermal_bridge_width 0.75)
+			(island_removal_mode 0)
+		)
+		(polygon
+			(pts
+				(arc
+					(start 189 60)
+					(mid 195 60)
+					(end 189 60)
+				)
+			)
+		)
+	)
+	(zone
+		(layers "F.Cu" "B.Cu")
+		(hatch edge 0.5)
+		(connect_pads
+			(clearance 0)
+		)
+		(min_thickness 0.25)
+		(keepout
+			(tracks allowed)
+			(vias allowed)
+			(pads allowed)
+			(copperpour not_allowed)
+			(footprints allowed)
+		)
+		(placement
+			(enabled no)
+			(sheetname "")
+		)
+		(fill
+			(thermal_gap 0.5)
+			(thermal_bridge_width 0.75)
+			(island_removal_mode 0)
+		)
+		(polygon
+			(pts
+				(arc
+					(start 189 152)
+					(mid 195 152)
+					(end 189 152)
+				)
+			)
+		)
