File: Active-PI/Active-PI.kicad_pcb (KiCad board)
At the start: 2 copper layers, 100 x 100 mm, 31 parts, among them U1 TL072

Commit message: PI
Parts:
- removed the C2 at (148.9, 107.6)
- removed JP2: Jumper_3_Open, Library:Jumper_1x03
- C2: renamed from C1; value 0.1uF -> 10nF
- R1: value 10k -> 100k
- moved C2 24.5 mm to (146.8, 107.6)
- moved R1 11.6 mm to (118.7, 117.3)
- moved JP1 11.4 mm to (135.7, 107.6)
- moved R2 3.00 mm to (133.1, 117.3)
- moved R3 3.00 mm to (133.1, 124.9)
- moved R4 3.00 mm to (157.2, 107.6)
- moved R5 3.00 mm to (166.7, 126.2)
- moved R6 3.00 mm to (174.5, 116.0)
- moved U1 3.00 mm to (151.4, 117.3)
Connections:
- C2 pad 1: Net-(JP1-A) -> Net-(JP1-B)
- C2 pad 2: Net-(JP1-B) -> Net-(C2-Pad2)
- R2 pad 1: Net-(JP1-B) -> Net-(JP1-A)
- R2 pad 2: Net-(C2-Pad2) -> Net-(JP1-B)
- U1 pad 2: Net-(JP1-B) -> Net-(JP1-A)
Routing:
- net Net-(JP1-B): track 49.4 -> 16.8 mm
- net Net-(D2-A): track 90.6 -> 71.3 mm
- net Net-(JP1-A): track 20.4 -> 37.0 mm
- net Net-(C2-Pad2): track 102.6 -> 92.4 mm
- net Net-(D1-K): track 33.1 -> 41.8 mm
- net GND: track 0.00 -> 7.07 mm
- net Net-(JP2-B): track 7.03 -> 0.00 mm
- net Net-(U1B--): track 32.0 -> 34.4 mm
- net Net-(R1-Pad1): track 62.4 -> 60.5 mm
- net Net-(U1B-+): track 18.4 -> 19.6 mm
- net Net-(R5-Pad2): track 52.3 -> 51.7 mm
Other:
- board text removed: "10k"
