File: Active-PI/Active-PI.kicad_sch (KiCad schematic)
At the start: 29 parts, among them U1 TL072

Commit message: PI
Parts:
- removed C2: 10nF, Capacitor_THT:C_Rect_L7.2mm_W2.5mm_P5.00mm, symbol Device:C
- removed JP1, JP2: Jumper_3_Open, Library:Jumper_1x03, symbol Jumper:Jumper_3_Open
Connections:
- net at R2.1, U1.2 (-): now also R1.2; no longer C1.2
- net at R4.1, TP5.1, U1.1: now also C1.2; no longer R2.2
- net at C1.1: now also R2.2; no longer R1.2
Other:
- moved on the sheet: C1, R1, R2, TP1, TP2

Commit message: PI
Parts:
- added JP1: Jumper_3_Open, Library:Jumper_1x03, symbol Jumper:Jumper_3_Open
- C2: renamed from C1; value 0.1uF -> 10nF; TME R82DC3100DQ50J -> R82EC2100AA50J
- R1: value 10k -> 100k
Connections:
- net at R1.2, R2.1, U1.2 (-): now also JP1.1 (A), JP1.2 (C)
- net at C2.1, R2.2: now also JP1.3 (B)
Other:
- moved on the sheet: C2
